Commit message: add gripper

File: ur_moveit_config/srdf/ur.srdf.xacro (robot description, xacro)
@@ -5,5 +5,6 @@
   <!-- parameters -->
   <xacro:arg name="prefix" default="" />
+  <xacro:arg name="with_gripper" default="true"/>
   <xacro:include filename="$(find ur_moveit_config)/srdf/ur_macro.srdf.xacro"/>
-  <xacro:ur_srdf name="$(arg name)" prefix="$(arg prefix)"/>
+  <xacro:ur_srdf name="$(arg name)" prefix="$(arg prefix)" with_gripper="$(arg with_gripper)" gripper_name="schunk"/>
 </robot>

File: ur_moveit_config/srdf/ur_macro.srdf.xacro (robot description, xacro)
@@ -5,5 +5,5 @@
     A URDF file must exist for this robot as well, where the joints and the links that are referenced are defined
 -->
-  <xacro:macro name="ur_srdf" params="name prefix">
+  <xacro:macro name="ur_srdf" params="name prefix with_gripper:=false gripper_name">
     <!--GROUPS - Representation of a set of joints and links. This can be useful for specifying DOF to plan for, defining arms, end effectors, etc-->
     <!--LINKS - When a link is specified, the parent joint of that link (if it exists) is automatically included-->
@@ -11,33 +11,44 @@
     <!--CHAINS - When a chain is specified, all the links along the chain (including endpoints) are included in the group. Additionally, all the joints that are parents to included links are also included. This means that joints along the chain and the parent joint of the base link are included in the group-->
     <!--SUBGROUPS - Groups can also be formed by referencing to already defined group names-->
-    <group name="${prefix}${name}_manipulator">
-      <chain base_link="${prefix}base_link" tip_link="${prefix}tool0" />
-    </group>
-    <!--GROUP STATES - Purpose - Define a named state for a particular group, in terms of joint values. This is useful to define states like 'folded arms'-->
-    <group_state name="${prefix}home" group="${prefix}${name}_manipulator">
-      <joint name="${prefix}elbow_joint" value="0" />
-      <joint name="${prefix}shoulder_lift_joint" value="-1.5707" />
-      <joint name="${prefix}shoulder_pan_joint" value="0" />
-      <joint name="${prefix}wrist_1_joint" value="0" />
-      <joint name="${prefix}wrist_2_joint" value="0" />
-      <joint name="${prefix}wrist_3_joint" value="0" />
-    </group_state>
-    <group_state name="${prefix}up" group="${prefix}${name}_manipulator">
-      <joint name="${prefix}elbow_joint" value="0" />
-      <joint name="${prefix}shoulder_lift_joint" value="-1.5707" />
-      <joint name="${prefix}shoulder_pan_joint" value="0" />
-      <joint name="${prefix}wrist_1_joint" value="-1.5707" />
-      <joint name="${prefix}wrist_2_joint" value="0" />
-      <joint name="${prefix}wrist_3_joint" value="0" />
-    </group_state>
-    <group_state name="${prefix}test_configuration" group="${prefix}${name}_manipulator">
-      <joint name="${prefix}elbow_joint" value="1.4" />
-      <joint name="${prefix}shoulder_lift_joint" value="-1.62" />
-      <joint name="${prefix}shoulder_pan_joint" value="1.54" />
-      <joint name="${prefix}wrist_1_joint" value="-1.2" />
-      <joint name="${prefix}wrist_2_joint" value="-1.6" />
-      <joint name="${prefix}wrist_3_joint" value="-0.11" />
-    </group_state>
+    <xacro:if value="${with_gripper}">
+        <group name="${prefix}${gripper_name}">
+          <joint name="${prefix}${gripper_name}_gripper_base_joint"/>
+          <joint name="${prefix}${gripper_name}_r_finger_joint"/>
+          <joint name="${prefix}${gripper_name}_l_finger_joint"/>
+          <joint name="${prefix}${gripper_name}_grasp_point"/>
+        </group>
+    </xacro:if>
+        <group name="${prefix}${name}_manipulator">
+            <chain base_link="${prefix}base_link" tip_link="${prefix}tool0" />
+        </group>
+        <!--GROUP STATES - Purpose - Define a named state for a particular group, in terms of joint values. This is useful to define states like 'folded arms'-->
+        <group_state name="${prefix}home" group="${prefix}${name}_manipulator">
+            <joint name="${prefix}elbow_joint" value="0" />
+            <joint name="${prefix}shoulder_lift_joint" value="-1.5707" />
+            <joint name="${prefix}shoulder_pan_joint" value="0" />
+            <joint name="${prefix}wrist_1_joint" value="0" />
+            <joint name="${prefix}wrist_2_joint" value="0" />
+        <joint name="${prefix}wrist_3_joint" value="0" />
+        </group_state>
+        <group_state name="${prefix}up" group="${prefix}${name}_manipulator">
+            <joint name="${prefix}elbow_joint" value="0" />
+            <joint name="${prefix}shoulder_lift_joint" value="-1.5707" />
+            <joint name="${prefix}shoulder_pan_joint" value="0" />
+            <joint name="${prefix}wrist_1_joint" value="-1.5707" />
+            <joint name="${prefix}wrist_2_joint" value="0" />
+            <joint name="${prefix}wrist_3_joint" value="0" />
+        </group_state>
+        <group_state name="${prefix}test_configuration" group="${prefix}${name}_manipulator">
+            <joint name="${prefix}elbow_joint" value="1.4" />
+            <joint name="${prefix}shoulder_lift_joint" value="-1.62" />
+            <joint name="${prefix}shoulder_pan_joint" value="1.54" />
+            <joint name="${prefix}wrist_1_joint" value="-1.2" />
+            <joint name="${prefix}wrist_2_joint" value="-1.6" />
+            <joint name="${prefix}wrist_3_joint" value="-0.11" />
+        </group_state>
     <!--END EFFECTOR - Purpose - Represent information about an end effector.-->
+    <xacro:if value="${with_gripper}">
+      <end_effector name="${gripper_name}" parent_link="${prefix}tool0" group="${prefix}${gripper_name}"/>
+    </xacro:if>
     <!--VIRTUAL JOINT - Purpose - this element defines a virtual joint between a robot link and an external frame of reference (considered fixed with respect to the robot)-->
     <!--DISABLE COLLISIONS - By default it is assumed that any link of the robot could potentially come into collision with any other link in the robot. This tag disables collision checking between a specified pair of links. -->
@@ -53,4 +64,54 @@
     <disable_collisions link1="${prefix}wrist_1_link" link2="${prefix}wrist_3_link" reason="Never" />
     <disable_collisions link1="${prefix}wrist_2_link" link2="${prefix}wrist_3_link" reason="Adjacent" />
+    <xacro:if value="${with_gripper}">
+      <disable_collisions link1="${gripper_name}_gripper_base_link" link2="${prefix}wrist_3_link" reason="Adjacent"/>
+      <disable_collisions link1="${gripper_name}_gripper_base_link" link2="${gripper_name}_l_finger_link" reason="Adjacent"/>
+      <disable_collisions link1="${gripper_name}_gripper_base_link" link2="${gripper_name}_r_finger_link" reason="Adjacent"/>
+      <disable_collisions link1="${gripper_name}_r_finger_link" link2="${gripper_name}_l_finger_link" reason="Adjacent"/>
+        <!-- <disable_collisions link1="${prefix}wrist_3_link" link2="${prefix}robotiq_85_base_link" reason="Adjacent" />
+        <disable_collisions link1="robotiq_85_base_link" link2="robotiq_85_left_finger_link" reason="Adjacent"/>
+        <disable_collisions link1="robotiq_85_base_link" link2="robotiq_85_left_finger_tip_link" reason="Adjacent"/>
+        <disable_collisions link1="robotiq_85_base_link" link2="robotiq_85_left_inner_knuckle_link" reason="Adjacent"/>
+        <disable_collisions link1="robotiq_85_base_link" link2="robotiq_85_left_knuckle_link" reason="Adjacent"/>
+        <disable_collisions link1="robotiq_85_base_link" link2="robotiq_85_right_finger_link" reason="Adjacent"/>
+        <disable_collisions link1="robotiq_85_base_link" link2="robotiq_85_right_finger_tip_link" reason="Adjacent"/>
+        <disable_collisions link1="robotiq_85_base_link" link2="robotiq_85_right_inner_knuckle_link" reason="Adjacent"/>
+        <disable_collisions link1="robotiq_85_base_link" link2="robotiq_85_right_knuckle_link" reason="Adjacent"/>
+        <disable_collisions link1="robotiq_85_left_finger_link" link2="robotiq_85_left_finger_tip_link" reason="Adjacent"/>
+        <disable_collisions link1="robotiq_85_left_finger_link" link2="robotiq_85_left_inner_knuckle_link" reason="Never"/>
+        <disable_collisions link1="robotiq_85_left_finger_link" link2="robotiq_85_left_knuckle_link" reason="Adjacent"/>
+        <disable_collisions link1="robotiq_85_left_finger_link" link2="robotiq_85_right_finger_link" reason="Adjacent"/>
+        <disable_collisions link1="robotiq_85_left_finger_link" link2="robotiq_85_right_finger_tip_link" reason="Adjacent"/>
+        <disable_collisions link1="robotiq_85_left_finger_link" link2="robotiq_85_right_inner_knuckle_link" reason="Adjacent"/>
+        <disable_collisions link1="robotiq_85_left_finger_link" link2="robotiq_85_right_knuckle_link" reason="Adjacent"/>
+        <disable_collisions link1="robotiq_85_left_finger_tip_link" link2="robotiq_85_left_inner_knuckle_link" reason="Default"/>
+        <disable_collisions link1="robotiq_85_left_finger_tip_link" link2="robotiq_85_left_knuckle_link" reason="Adjacent"/>
+        <disable_collisions link1="robotiq_85_left_finger_tip_link" link2="robotiq_85_right_finger_link" reason="Adjacent"/>
+        <disable_collisions link1="robotiq_85_left_finger_tip_link" link2="robotiq_85_right_finger_tip_link" reason="Adjacent"/>
+        <disable_collisions link1="robotiq_85_left_finger_tip_link" link2="robotiq_85_right_inner_knuckle_link" reason="Adjacent"/>
+        <disable_collisions link1="robotiq_85_left_finger_tip_link" link2="robotiq_85_right_knuckle_link" reason="Adjacent"/>
+        <disable_collisions link1="robotiq_85_left_inner_knuckle_link" link2="robotiq_85_left_knuckle_link" reason="Adjacent"/>
+        <disable_collisions link1="robotiq_85_left_inner_knuckle_link" link2="robotiq_85_right_finger_link" reason="Adjacent"/>
+        <disable_collisions link1="robotiq_85_left_inner_knuckle_link" link2="robotiq_85_right_finger_tip_link" reason="Adjacent"/>
+        <disable_collisions link1="robotiq_85_left_inner_knuckle_link" link2="robotiq_85_right_inner_knuckle_link" reason="Adjacent"/>
+        <disable_collisions link1="robotiq_85_left_inner_knuckle_link" link2="robotiq_85_right_knuckle_link" reason="Adjacent"/>
+        <disable_collisions link1="robotiq_85_left_knuckle_link" link2="robotiq_85_right_finger_link" reason="Adjacent"/>
+        <disable_collisions link1="robotiq_85_left_knuckle_link" link2="robotiq_85_right_finger_tip_link" reason="Adjacent"/>
+        <disable_collisions link1="robotiq_85_left_knuckle_link" link2="robotiq_85_right_inner_knuckle_link" reason="Adjacent"/>
+        <disable_collisions link1="robotiq_85_left_knuckle_link" link2="robotiq_85_right_knuckle_link" reason="Adjacent"/>
+        <disable_collisions link1="robotiq_85_right_finger_link" link2="robotiq_85_right_finger_tip_link" reason="Adjacent"/>
+        <disable_collisions link1="robotiq_85_right_finger_link" link2="robotiq_85_right_inner_knuckle_link" reason="Adjacent"/>
+        <disable_collisions link1="robotiq_85_right_finger_link" link2="robotiq_85_right_knuckle_link" reason="Adjacent"/>
+        <disable_collisions link1="robotiq_85_right_finger_tip_link" link2="robotiq_85_right_inner_knuckle_link" reason="Default"/>
+        <disable_collisions link1="robotiq_85_right_finger_tip_link" link2="robotiq_85_right_knuckle_link" reason="Adjacent"/>
+        <disable_collisions link1="robotiq_85_right_inner_knuckle_link" link2="robotiq_85_right_knuckle_link" reason="Adjacent"/>
+        <disable_collisions link1="robotiq_85_base_link" link2="rgbd_camera" reason="Adjacent"/> -->
+        <!-- <disable_collisions link1="${prefix}forearm_link" link2="robotiq_85_left_finger_link" reason="Never"/>
+        <disable_collisions link1="${prefix}forearm_link" link2="robotiq_85_right_finger_link" reason="Never"/>
+        <disable_collisions link1="${prefix}forearm_link" link2="robotiq_85_right_finger_tip_link" reason="Never"/>
+        <disable_collisions link1="${prefix}forearm_link" link2="robotiq_85_left_finger_tip_link" reason="Never"/>
+        <disable_collisions link1="${prefix}forearm_link" link2="robotiq_85_left_knuckle_link" reason="Never"/>
+        <disable_collisions link1="${prefix}forearm_link" link2="robotiq_85_right_knuckle_link" reason="Never"/> -->
+    </xacro:if>
   </xacro:macro>
 </robot>
