Commit message: srdf with gripper xacro edit

File: ur_moveit_config/srdf/ur_macro.srdf.xacro (robot description, xacro)
@@ -12,14 +12,18 @@
     <!--SUBGROUPS - Groups can also be formed by referencing to already defined group names-->
     <xacro:if value="${with_gripper}">
+        <group name="${prefix}${name}_manipulator">
+            <chain base_link="${prefix}base_link" tip_link="${prefix}${gripper_name}_grasp_point" />
+        </group>
         <group name="${prefix}${gripper_name}">
           <joint name="${prefix}${gripper_name}_gripper_base_joint"/>
           <joint name="${prefix}${gripper_name}_r_finger_joint"/>
           <joint name="${prefix}${gripper_name}_l_finger_joint"/>
-          <joint name="${prefix}${gripper_name}_grasp_point"/>
         </group>
     </xacro:if>
+    <xacro:unless value="${with_gripper}">
         <group name="${prefix}${name}_manipulator">
             <chain base_link="${prefix}base_link" tip_link="${prefix}tool0" />
         </group>
+    </xacro:unless>
         <!--GROUP STATES - Purpose - Define a named state for a particular group, in terms of joint values. This is useful to define states like 'folded arms'-->
         <group_state name="${prefix}home" group="${prefix}${name}_manipulator">
@@ -49,5 +53,5 @@
     <!--END EFFECTOR - Purpose - Represent information about an end effector.-->
     <xacro:if value="${with_gripper}">
-      <end_effector name="${gripper_name}" parent_link="${prefix}tool0" group="${prefix}${gripper_name}"/>
+      <!-- <end_effector name="${gripper_name}" parent_link="${prefix}tool0" group="${prefix}${gripper_name}"/> -->
     </xacro:if>
     <!--VIRTUAL JOINT - Purpose - this element defines a virtual joint between a robot link and an external frame of reference (considered fixed with respect to the robot)-->
